Commit message: Gazebo added

File: description/robot.urdf.xacro (robot description, xacro)
@@ -2,3 +2,4 @@
 <robot xmlns:xacro="http://www.ros.org/wiki/xacro" name="robot">
 <xacro:include filename="robot_core.xacro"/>
+<xacro:include filename="gazebo_control.xacro" />
 </robot>

File: description/robot_core.xacro (robot description, xacro)
@@ -45,4 +45,7 @@
         </xacro:inertial_box>
     </link>
+    <gazebo reference="chassis">
+        <material>Gazebo/White</material>
+    </gazebo>
     <!-- LEFT WHEEL -->
     <joint name="left_wheel_joint" type="continuous">
@@ -68,8 +71,11 @@
         </xacro:inertial_cylinder>
     </link>
+    <gazebo reference="left_wheel">
+        <material>Gazebo/Blue</material>
+    </gazebo>
     <joint name="right_wheel_joint" type="continuous">
         <parent link="base_link"/>
         <child link="right_wheel"/>
-        <origin xyz="0 -0.22 0" rpy="-1.57079632679 0 0" />
+        <origin xyz="0 -0.22 0" rpy="1.57079632679 0 0" />
         <axis xyz="0 0 -1"/>
     </joint>
@@ -90,4 +96,7 @@
         </xacro:inertial_cylinder>
     </link>
+    <gazebo reference="right_wheel">
+        <material>Gazebo/Blue</material>
+    </gazebo>
     <!-- CASTER WHEELs -->
     <joint name="caster_wheel_joint_left" type="fixed">
@@ -112,4 +121,7 @@
         </xacro:inertial_sphere>
     </link>
+    <gazebo reference="caster_wheel_left">
+        <material>Gazebo/Blue</material>
+    </gazebo>
     <joint name="caster_wheel_right_joint" type="fixed">
         <parent link="chassis"/>
@@ -133,3 +145,6 @@
         </xacro:inertial_sphere>
     </link>
+    <gazebo reference="caster_wheel_right">
+        <material>Gazebo/Blue</material>
+    </gazebo>
 </robot>
